File: pcb/EFM8_USB_Debug_Adapter/B1/Connectors.kicad_sch (KiCad schematic)
At the start: 36 parts, among them J100 EFM8_IDC_Debug_Header_Horizon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, J110 2137160001, J111 TTL-232R_Header_Horizontal, J120 31230102, J130 EFM8_USB_8-Bit_Debug_Header_H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, J131 Header_01x02_Wurth_61300211121, M110 USB_Light_Pipe, M120 PSU_Light_Pipe, M130 DBG8_Light_Pipe, Q110 SI3443CDV-T1-GE3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

Commit message: Update resistor values, LED colors
Parts:
- D120, D121: value 150080SS75000 -> 150080GS75000; symbol LED_User:150080SS75000 -> LED_User:150080GS75000; Info Red -> Green; SPN 732-4985-1-ND -> 732-4983-1-ND
- D130, D131: value 150080SS75000 -> 150080BS75000; symbol LED_User:150080SS75000 -> LED_User:150080BS75000; Info Red -> Blue; SPN 732-4985-1-ND -> 732-4982-1-ND
- R112, R115: value 2k,0603 -> 680R,0603; symbol Resistor_User:2k,0603 -> Resistor_User:680R,0603; Resistance 2k -> 680R
- R113, R121, R131: value 75k,0603 -> 47k,0603; symbol Resistor_User:75k,0603 -> Resistor_User:47k,0603; Resistance 75k -> 47k
- R120, R123: value 2k,0603 -> 1k,0603; symbol Resistor_User:2k,0603 -> Resistor_User:1k,0603; Resistance 2k -> 1k
- R130, R133: value 2k,0603 -> 470R,0603; symbol Resistor_User:2k,0603 -> Resistor_User:470R,0603; Resistance 2k -> 470R
Changed lines of the file:
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@@
 	)
 	(symbol
-		(lib_id "LED_User:150080SS75000")
+		(lib_id "LED_User:150080GS75000")
 		(at 124.46 87.63 90)
 		(unit 1)
@@
 			)
 		)
-		(property "Value" "150080SS75000"
-			(at 119.38 92.71 0)
+		(property "Value" "150080GS75000"
+			(at 127.254 88.646 0)
 			(effects
 				(font
@@
 			)
 		)
-		(property "Datasheet" "https://www.we-online.com/katalog/datasheet/150080SS75000.pdf"
+		(property "Datasheet" "https://www.we-online.com/katalog/datasheet/150080GS75000.pdf"
 			(at 124.46 88.9 0)
 			(effects
@@
 			)
 		)
-		(property "Description" ""
+		(property "Description" "Top View SMD LED, Clear Green, 0805"
 			(at 124.46 87.63 0)
 			(effects
@@
 			)
 		)
-		(property "SPN" "732-4985-1-ND"
+		(property "SPN" "732-4983-1-ND"
 			(at 134.62 90.17 0)
 			(effects
@@
 			)
 		)
-		(property "Info" "Red"
-			(at 129.54 90.17 90)
+		(property "Info" "Green"
+			(at 129.54 88.9 0)
 			(effects
 				(font
@@
 	)
 	(symbol
-		(lib_id "Resistor_User:2k,0603")
+		(lib_id "Resistor_User:470R,0603")
 		(at 101.6 147.32 0)
 		(unit 1)
@@
 			)
 		)
-		(property "Value" "2k,0603"
+		(property "Value" "470R,0603"
 			(at 103.505 144.78 0)
 			(effects
@@
 			)
 		)
-		(property "Description" ""
+		(property "Description" "Resistor, 0603"
 			(at 101.6 147.32 0)
 			(effects
@@
 			)
 		)
-		(property "Resistance" "2k"
+		(property "Resistance" "470R"
 			(at 104.14 148.5899 0)
 			(effects
@@
 	)
 	(symbol
-		(lib_id "LED_User:150080SS75000")
+		(lib_id "LED_User:150080BS75000")
 		(at 124.46 138.43 90)
 		(unit 1)
@@
 			)
 		)
-		(property "Value" "150080SS75000"
+		(property "Value" "150080BS75000"
 			(at 127.254 139.446 0)
 			(effects
@@
 			)
 		)
-		(property "Datasheet" "https://www.we-online.com/katalog/datasheet/150080SS75000.pdf"
+		(property "Datasheet" "https://www.we-online.com/katalog/datasheet/150080BS75000.pdf"
 			(at 124.46 139.7 0)
 			(effects
@@
 			)
 		)
-		(property "Description" ""
+		(property "Description" "Top View SMD LED, Clear Blue, 0805"
 			(at 124.46 138.43 0)
 			(effects
@@
 			)
 		)
-		(property "SPN" "732-4985-1-ND"
+		(property "SPN" "732-4982-1-ND"
 			(at 134.62 140.97 0)
 			(effects
@@
 			)
 		)
-		(property "Info" "Red"
+		(property "Info" "Blue"
 			(at 129.54 139.7 0)
 			(effects
@@
 	)
 	(symbol
-		(lib_id "LED_User:150080SS75000")
+		(lib_id "LED_User:150080BS75000")
 		(at 101.6 138.43 90)
 		(unit 1)
@@
 			)
 		)
-		(property "Value" "150080SS75000"
+		(property "Value" "150080BS75000"
 			(at 104.394 139.446 0)
 			(effects
@@
 			)
 		)
-		(property "Datasheet" "https://www.we-online.com/katalog/datasheet/150080SS75000.pdf"
+		(property "Datasheet" "https://www.we-online.com/katalog/datasheet/150080BS75000.pdf"
 			(at 101.6 139.7 0)
 			(effects
@@
 			)
 		)
-		(property "Description" ""
+		(property "Description" "Top View SMD LED, Clear Blue, 0805"
 			(at 101.6 138.43 0)
 			(effects
@@
 			)
 		)
-		(property "SPN" "732-4985-1-ND"
+		(property "SPN" "732-4982-1-ND"
 			(at 111.76 140.97 0)
 			(effects
@@
 			)
 		)
-		(property "Info" "Red"
+		(property "Info" "Blue"
 			(at 106.68 139.7 0)
 			(effects
@@
 	)
 	(symbol
-		(lib_id "LED_User:150080SS75000")
+		(lib_id "LED_User:150080GS75000")
 		(at 101.6 87.63 90)
 		(unit 1)
@@
 			)
 		)
-		(property "Value" "150080SS75000"
-			(at 96.52 92.71 0)
+		(property "Value" "150080GS75000"
+			(at 104.394 88.646 0)
 			(effects
 				(font
@@
 			)
 		)
-		(property "Datasheet" "https://www.we-online.com/katalog/datasheet/150080SS75000.pdf"
+		(property "Datasheet" "https://www.we-online.com/katalog/datasheet/150080GS75000.pdf"
 			(at 101.6 88.9 0)
 			(effects
@@
 			)
 		)
-		(property "Description" ""
+		(property "Description" "Top View SMD LED, Clear Green, 0805"
 			(at 101.6 87.63 0)
 			(effects
@@
 			)
 		)
-		(property "SPN" "732-4985-1-ND"
+		(property "SPN" "732-4983-1-ND"
 			(at 111.76 90.17 0)
 			(effects
@@
 			)
 		)
-		(property "Info" "Red"
-			(at 106.68 90.17 90)
+		(property "Info" "Green"
+			(at 106.68 88.9 0)
 			(effects
 				(font
@@
 	)
 	(symbol
-		(lib_id "Resistor_User:75k,0603")
+		(lib_id "Resistor_User:47k,0603")
 		(at 148.59 53.34 0)
 		(unit 1)
@@
 			)
 		)
-		(property "Value" "75k,0603"
+		(property "Value" "47k,0603"
 			(at 150.495 50.8 0)
 			(effects
@@
 			)
 		)
-		(property "Resistance" "75k"
+		(property "Resistance" "47k"
 			(at 151.13 54.6099 0)
 			(effects
@@
 	)
 	(symbol
-		(lib_id "Resistor_User:2k,0603")
+		(lib_id "Resistor_User:470R,0603")
 		(at 124.46 147.32 0)
 		(unit 1)
@@
 			)
 		)
-		(property "Value" "2k,0603"
+		(property "Value" "470R,0603"
 			(at 126.365 144.78 0)
 			(effects
@@
 			)
 		)
-		(property "Description" ""
+		(property "Description" "Resistor, 0603"
 			(at 124.46 147.32 0)
 			(effects
@@
 			)
 		)
-		(property "Resistance" "2k"
+		(property "Resistance" "470R"
 			(at 127 148.5899 0)
 			(effects
@@
 	)
 	(symbol
-		(lib_id "Resistor_User:75k,0603")
+		(lib_id "Resistor_User:47k,0603")
 		(at 148.59 113.03 0)
 		(unit 1)
@@
 			)
 		)
-		(property "Value" "75k,0603"
+		(property "Value" "47k,0603"
 			(at 150.495 110.49 0)
 			(effects
@@
 			)
 		)
-		(property "Resistance" "75k"
+		(property "Resistance" "47k"
 			(at 151.13 114.2999 0)
 			(effects
@@
 	)
 	(symbol
-		(lib_id "Resistor_User:2k,0603")
+		(lib_id "Resistor_User:680R,0603")
 		(at 124.46 36.83 0)
 		(unit 1)
@@
 			)
 		)
-		(property "Value" "2k,0603"
+		(property "Value" "680R,0603"
 			(at 126.365 34.29 0)
 			(effects
@@
 			)
 		)
-		(property "Description" ""
+		(property "Description" "Resistor, 0603"
 			(at 124.46 36.83 0)
 			(effects
@@
 			)
 		)
-		(property "Resistance" "2k"
+		(property "Resistance" "680R"
 			(at 127 38.0999 0)
 			(effects
@@
 	)
 	(symbol
-		(lib_id "Resistor_User:2k,0603")
+		(lib_id "Resistor_User:1k,0603")
 		(at 124.46 96.52 0)
 		(unit 1)
@@
 			)
 		)
-		(property "Value" "2k,0603"
+		(property "Value" "1k,0603"
 			(at 126.365 93.98 0)
 			(effects
@@
 			)
 		)
-		(property "Description" ""
+		(property "Description" "Resistor, 0603"
 			(at 124.46 96.52 0)
 			(effects
@@
 			)
 		)
-		(property "Resistance" "2k"
+		(property "Resistance" "1k"
 			(at 127 97.7899 0)
 			(effects
@@
 	)
 	(symbol
-		(lib_id "Resistor_User:75k,0603")
+		(lib_id "Resistor_User:47k,0603")
 		(at 148.59 163.83 0)
 		(unit 1)
@@
 			)
 		)
-		(property "Value" "75k,0603"
+		(property "Value" "47k,0603"
 			(at 150.495 161.29 0)
 			(effects
@@
 			)
 		)
-		(property "Resistance" "75k"
+		(property "Resistance" "47k"
 			(at 151.13 165.0999 0)
 			(effects
@@
 	)
 	(symbol
-		(lib_id "Resistor_User:2k,0603")
+		(lib_id "Resistor_User:1k,0603")
 		(at 101.6 96.52 0)
 		(unit 1)
@@
 			)
 		)
-		(property "Value" "2k,0603"
+		(property "Value" "1k,0603"
 			(at 103.505 93.98 0)
 			(effects
@@
 			)
 		)
-		(property "Description" ""
+		(property "Description" "Resistor, 0603"
 			(at 101.6 96.52 0)
 			(effects
@@
 			)
 		)
-		(property "Resistance" "2k"
+		(property "Resistance" "1k"
 			(at 104.14 97.7899 0)
 			(effects
@@
 	)
 	(symbol
-		(lib_id "Resistor_User:2k,0603")
+		(lib_id "Resistor_User:680R,0603")
 		(at 101.6 36.83 0)
 		(unit 1)
@@
 			)
 		)
-		(property "Value" "2k,0603"
+		(property "Value" "680R,0603"
 			(at 103.505 34.29 0)
 			(effects
@@
 			)
 		)
-		(property "Description" ""
+		(property "Description" "Resistor, 0603"
 			(at 101.6 36.83 0)
 			(effects
@@
 			)
 		)
-		(property "Resistance" "2k"
+		(property "Resistance" "680R"
 			(at 104.14 38.0999 0)
 			(effects
